File: pcb/Orion-Control-Board/Orion-Control-Board.kicad_sch (KiCad schematic)
At the start: 50 parts, among them J1 CORTEX_DEBUG_SWD_UART, J2 STLINK_SWD_JTAG_20POS, J3 USB C 2.0 Female, J4 GPIO_DEBUG_HEADER, U1 FT232RL, U2 USBLC6-2SC6, U3 LM66100, U4 LM66100, U5 LM2596_ADJ_BUCK

Commit message: Design IMU, Voltage Sensor, and Driver circuits
Parts:
- removed BZ: Buzzer, symbol Device:Buzzer
- removed C6: 100nF, Capacitor_SMD:C_0402_1005Metric, symbol Device:C
- removed D4: RX, LED_SMD:LED_0805_2012Metric, symbol Device:LED
- removed D5: RPI_ON, AA_Custom_Components:LED_SS_1206_3216Metric_Pad1.42x1.75mm_HandSolder, symbol Device:LED
- removed D6: USER_LED, AA_Custom_Components:LED_SS_1206_3216Metric_Pad1.42x1.75mm_HandSolder, symbol Device:LED
- removed F1: 6V 500mA Fuse, Fuse:Fuse_0603_1608Metric, symbol Device:Fuse
- removed FB1: 100Ω@100MHz, Inductor_SMD:L_0805_2012Metric, symbol Device:FerriteBead
- removed J: MPU6050_IMU, symbol AA_Custom_Components:MPU6050_IMU
- removed J1: CORTEX_DEBUG_SWD_UART, AA_Custom_Components:SAMTEC_FTSH-105-XX-X-DV, symbol AA_Custom_Components:CORTEX_DEBUG_SMD_UART
- removed J2: STLINK_SWD_JTAG_20POS, AA_Custom_Components:SULLINS_SFH11-PBPC-D10-ST-BK, symbol AA_Custom_Components:STLINK_SWD_JTAG_20Pos
- removed J3: USB C 2.0 Female, Connector_USB:USB_C_Receptacle_HRO_TYPE-C-31-M-12, symbol AA_Custom_Components:USB_C_Receptacle_USB2.0_16P
- removed JP2: Jumper_2_Open, AA_Custom_Components:R_SS_Axial_DIN0207_L6.3mm_D2.5mm_P10.16mm_Horizontal, symbol Jumper:Jumper_2_Open
- removed N1, N2: CENTER_POS, AA_Custom_Components:Polarity_Center_Positive_7.5mm_SilkScreen, symbol Mechanical:Housing
- removed U1: FT232RL, Package_SO:SSOP-28_5.3x10.2mm_P0.65mm, symbol Interface_USB:FT232RL
- removed U2: USBLC6-2SC6, Package_TO_SOT_SMD:SOT-23-6, symbol Power_Protection:USBLC6-2SC6
- removed U3, U4: LM66100, Package_TO_SOT_SMD:SOT-363_SC-70-6, symbol AA_Custom_Components:LM66100
- removed U5: LM2596_ADJ_BUCK, symbol AA_Custom_Components:LM2596_ADJ_BUCK
- added C10, C9: 22pF, Capacitor_SMD:C_0603_1608Metric, symbol Device:C
- added C7: 100nF, Capacitor_SMD:C_0603_1608Metric, symbol Device:C
- added C8: 1uF, Capacitor_SMD:C_0603_1608Metric, symbol Device:C
- added J3: Keyed Connector 20 pos, AA_Custom_Components:SULLINS_SFH11-PBPC-D10-ST-BK, symbol AA_Custom_Components:20PosKeyedMale
- added JP3: PCA Jumper, AA_Custom_Components:R_SS_Axial_DIN0207_L6.3mm_D2.5mm_P10.16mm_Horizontal, symbol Jumper:Jumper_2_Open
- added R14, R15, R16, R17, R18, R19: 220, Resistor_SMD:R_0603_1608Metric, symbol Device:R
- added R20, R21, R22: 4.7k, Resistor_SMD:R_0603_1608Metric, symbol Device:R
- added R23, R24, R25, R26, R27, R28, R33, R34, R35, R36: 10k, Resistor_SMD:R_0603_1608Metric, symbol Device:R
- added U1, U2, U4: INA3221, Package_DFN_QFN:Texas_RGV0016A_VQFN-16-1EP_4x4mm_P0.65mm_EP2.1x2.1mm, symbol AA_Custom_Components:INA3221
- added U3: PCA9685_PWM_SERVO_DRIVER_IC, Silicon-Standard:TSSOP-28_4MM, symbol AA_Custom_Components:PCA9685_PWM_SERVO_DRIVER_IC
- added U5: DFR0753_5V_BUCK, symbol AA_Custom_Components:DFR0753_5V_BUCK
- added U6: BNO055, Package_LGA:LGA-28_5.2x3.8mm_P0.5mm, symbol AA_Custom_Components:BNO055
- added Y1: 32.768 kHz, CRYSTAL-SMD-3.2X1.5MM, symbol AA_Custom_Components:CRYSTAL-32.768Khz
- C1: value 100nF -> 10uF; footprint Capacitor_SMD:C_0402_1005Metric -> Capacitor_SMD:C_0603_1608Metric; JLCPCB Part # C1525 -> C96446
- C2, C5: footprint Capacitor_SMD:C_0402_1005Metric -> Capacitor_SMD:C_0603_1608Metric; JLCPCB Part # C1525 -> C14663
- C3: value 4.7uF -> 100nF; footprint Capacitor_SMD:C_0805_2012Metric -> Capacitor_SMD:C_0603_1608Metric; JLCPCB Part # C1779 -> C14663
- C4: value 10nF -> 100nF; footprint Capacitor_SMD:C_0402_1005Metric -> Capacitor_SMD:C_0603_1608Metric; JLCPCB Part # C15195 -> C14663
- D1: value 3.3V -> 5V Buck; footprint LED_SMD:LED_0603_1608Metric -> LED_SMD:LED_0805_2012Metric; JLCPCB Part # C2290 -> C2297; Manufacturer Part # KT-0603W -> KT-0805G
- D2: value 5V -> 3.3V STM32
- D3: value TX -> DEBUG STM32
- JP1: value Jumper_2_Open -> BNO Jumper
- N4: value CENTER_POS -> ORION LOGO
- R1, R3: value 100k -> 220; footprint Resistor_SMD:R_0402_1005Metric -> Resistor_SMD:R_0603_1608Metric; JLCPCB Part # C25741 -> C25804
- R10, R11: value 100 -> 220; footprint Resistor_SMD:R_0402_1005Metric -> Resistor_SMD:R_0603_1608Metric; JLCPCB Part # C25076 -> C25804
- R12: value 220 -> 10k; footprint AA_Custom_Components:R_SS_Axial_DIN0207_L6.3mm_D2.5mm_P10.16mm_Horizontal -> Resistor_SMD:R_0603_1608Metric; JLCPCB Part # (none) -> C25804
- R13: value 22 -> 10k; footprint AA_Custom_Components:R_SS_Axial_DIN0207_L6.3mm_D2.5mm_P10.16mm_Horizontal -> Resistor_SMD:R_0603_1608Metric; JLCPCB Part # (none) -> C25804
- R2: value 100k -> 10k; footprint Resistor_SMD:R_0402_1005Metric -> Resistor_SMD:R_0603_1608Metric; JLCPCB Part # C25741 -> C25804
- R4: value 100 -> 470; footprint Resistor_SMD:R_0402_1005Metric -> Resistor_SMD:R_0603_1608Metric; JLCPCB Part # C25076 -> C23179
- R5, R6: value 680 -> 75; JLCPCB Part # C23228 -> C4275
- R7: value 680 -> 4.7k; JLCPCB Part # C23228 -> C23162
- R8, R9: value 5k1 -> 220; footprint Resistor_SMD:R_0402_1005Metric -> Resistor_SMD:R_0603_1608Metric; JLCPCB Part # C25905 -> C25804
Connections:
- net +3.3VP is gone; now on net +3.3V: JP1.2 (B)
- net +3V3 is gone; now on an unnamed net: JP1.1 (A)
- net TXLED is gone; now on net GND: R6.2
- net +3.3V: now also C3.1, C4.1, C5.1, D2.2 (A), R12.2, R13.2, R7.1, JP3.2 (B), R20.1, R21.1, R22.1, R23.2, R24.2, R25.2, R26.2, R27.2, R28.2, R33.2, R34.2, R35.2, R36.2, U1.16 (VPU), U1.4 (VS), U1.5 (A0), U2.16 (VPU), U2.4 (VS), U4.16 (VPU), U4.4 (VS), U6.11 (~{RESET}), U6.4 (~{BOOT_LOAD_PIN}); no longer D1.2 (A), R1.1, R2.1
- net +5V: now also D1.2 (A), U5.3 (VOUT); no longer C3.1, C5.1, D2.2 (A), D3.2 (A)
- net GND: now also C1.1, R2.1, C10.2, C7.2, C8.2, C9.1, J3.19, U1.17 (THERMALPAD), U1.3 (GND), U2.17 (THERMALPAD), U2.3 (GND), U3.1 (A0), U3.14 (VSS), U3.2 (A1), U3.24 (A5), U3.25 (EXTCLK), U3.3 (A2), U3.4 (A3), U3.5 (A4), U4.17 (THERMALPAD), U4.3 (GND), U5.2 (GND), U6.17 (I2CADDR), U6.18 (COM2), U6.2 (GND), U6.25 (GNDIO), U6.5 (PS1), U6.6 (PS0); no longer C1.2, R12.2, R13.2, R3.2, R8.2, R9.2
- net at R12.1: now also U1.8 (WARNING)
- net at R10.1: now also U3.10 (CH4)
- net at C2.2: now also C7.1, U6.28 (VDDIO), U6.3 (VDD)
- net at R11.1: now also U3.11 (CH5)
- net at R13.1: now also U1.9 (CRITICAL)
- net at R8.1: now also U3.8 (CH2)
- net at R9.1: now also U3.9 (CH3)
- net RXLED renamed SDA_{1}
- net SDA_{1}: now also U3.27 (SDA)
- net RX_{STM32} renamed PWM4
- net PWM4: now also J3.5
- net SWCLK: no longer names the net of R3.1
- net SWCLK: now also U3.7 (CH1)
- net SWDIO: no longer names the net of R2.2
- net SWDIO: now also U3.23 (~{OE})
- net TX_{STM32} renamed PWM5
- net PWM5: now also J3.6
- net USER_LED_BUZZER renamed BUZZER
- net nReset renamed PWM0
- net PWM0: now also J3.1; no longer C1.1
- new net: R36.1, U2.13 (TC)
- new net: R1.1, U3.6 (CH0)
- new net: R25.1, U4.10 (PV)
- new net: R28.1, U4.13 (TC)
- new net: R27.1, U4.8 (WARNING)
- new net: R26.1, U4.9 (CRITICAL)
- new net: C1.2, JP3.1 (A), U3.28 (VDD)
- new net: R18.2, U3.17 (CH10)
- new net: C9.2, U6.27 (XIN32), Y1.P$2 (2)
- new net: R35.1, U2.8 (WARNING)
- new net: R14.1, U3.12 (CH6)
- new net: R23.1, U1.13 (TC)
- new net: C10.1, U6.26 (XOUT32), Y1.P$1 (1)
- new net: C8.1, U6.9 (CAP)
- new net: R34.1, U2.9 (CRITICAL)
- new net: R16.2, U3.15 (CH8)
- new net: R24.1, U1.10 (PV)
- new net: R19.2, U3.18 (CH11)
- new net: R17.2, U3.16 (CH9)
- new net: R33.1, U2.10 (PV)
- new net: R15.1, U3.13 (CH7)
- new net 2S_BATT_FRONT_CELL1: J3.18, U1.11 (IN-1)
- new net 2S_BATT_FRONT_CELL2: J3.20, U1.14 (IN-2), U5.1 (VIN)
- new net 2S_BATT_REAR_CELL1: J3.14, U2.11 (IN-1)
- new net 2S_BATT_REAR_CELL2: J3.16, U2.14 (IN-2)
- new net 3S_BATT_CELL1: J3.13, U4.11 (IN-1)
- new net 3S_BATT_CELL2: J3.15, U4.14 (IN-2)
- new net 3S_BATT_CELL3: J3.17, U4.1 (IN-3)
- new net LED_DEBUG: D3.2 (A)
- new net PWM1: J3.2, R3.2
- new net PWM10: J3.11, R18.1
- new net PWM11: J3.12, R19.1
- new net PWM2: J3.3, R8.2
- new net PWM3: J3.4, R9.2
- new net PWM6: J3.7, R14.2
- new net PWM7: J3.8, R15.2
- new net PWM8: J3.9, R16.1
- new net PWM9: J3.10, R17.1
- new net SCL_{1}: R20.2, U3.26 (SCL)
- new net SCL_{2}: R22.2, U1.6 (SCL), U2.6 (SCL), U4.5 (A0), U4.6 (SCL), U6.19 (COM1)
- new net SDA_{2}: R21.2, U1.7 (SDA), U2.5 (A0), U2.7 (SDA), U4.7 (SDA), U6.20 (COM0)
- no-connect marks 14 -> 18
Other:
- note added: "12-bit PWM driver I2C Addr: 0x40"
- note added: "Battery Voltage Monitors"
- note added: "Buck"
- note added: "I2C Addr: 0x28"
- note added: "I2C Addr: 0x41"
- note added: "I2C Addr: 0x42"
- note added: "I2C Addr: 0x43"
- note added: "I2C Pullups"
- note added: "IMU"
- note added: "LEDs"
- note added: "OpenDrain Outputs can generally be left unconnected. Here, added 10k pullups anyways in case IC uses requires it internally"
- note added: "Power-board Connection"
- note added: "Select I2C mode"
- note added: "Servo Driver"
- note added: "TODO: add caps?"
- note added: "Try to use 0603 (1608m) everywhere. Not smaller."
- note added: "Unsure if Jetson (I2C1) has pullup resistors TODO: Could add extra DNP resistors to change speed?"
- note removed: "BLUE"
- note removed: "DNP"
- note removed: "EMI"
- note removed: "ESD"
- note removed: "INDICATOR LED"
- note removed: "No reverse polarity protection, since USB is standardized"
- note removed: "Note: Connect these jumpers if not using LDO"
- note removed: "PER FTDI"
- note removed: "POWER JUMPERS"
- note removed: "Reverse Current Protection - Blocks Debug connector from accepting power input"
- note removed: "STLINK"
- note removed: "USB-UART-Interface"
- note removed: "V_{ref} is I/O reference voltage from external STM32 PCB for the STLINK and FTDI UART"
- note removed: "WHITE"
- moved on the sheet: BZ1, D2, D3, H1, H2, H3, H4, J4, JP1, N3, N4, R5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

Commit message: Add lipo tester and LTC extender
Parts:
- removed C4, C5: 100nF, Capacitor_SMD:C_0603_1608Metric, symbol Device:C
- removed R20, R21, R22: 4.7k, Resistor_SMD:R_0603_1608Metric, symbol Device:R
- added C1, C10, C9: 100nF, Capacitor_SMD:C_0603_1608Metric, symbol Device:C
- added J2: 5V Select Socket, Connector_PinSocket_2.54mm:PinSocket_1x03_P2.54mm_Vertical, symbol dk_Rectangular-Connectors-Headers-Male-Pins:640456-3
- added J3: 5V Select Jumper, digikey-footprints:PinHeader_1x3_P2.54_Drill1.1mm, symbol dk_Rectangular-Connectors-Headers-Male-Pins:640456-3
- added J5, J6, J7: LIPO_VOLTAGE_ALARM, AA_Custom_Components:LIPO_VOLTAGE_ALARM, symbol AA_Custom_Components:LIPO_VOLTAGE_ALARM
- added JP1: I2C Extend Jumper, Connector_PinHeader_2.54mm:PinHeader_1x02_P2.54mm_Vertical, symbol Jumper:Jumper_2_Open
- added JP4: I2C Select SDA, Connector_PinHeader_2.54mm:PinHeader_1x03_P2.54mm_Vertical, symbol Jumper:Jumper_3_Bridged12
- added JP5: I2C Select SCL, Connector_PinHeader_2.54mm:PinHeader_1x03_P2.54mm_Vertical, symbol Jumper:Jumper_3_Bridged12
- added JP6: V_{Sense1} Jumper, Connector_PinHeader_2.54mm:PinHeader_1x02_P2.54mm_Vertical, symbol Jumper:Jumper_2_Open
- added JP7: V_{Sense2} Jumper, Connector_PinHeader_2.54mm:PinHeader_1x02_P2.54mm_Vertical, symbol Jumper:Jumper_2_Open
- added JP8: V_{Sense3} Jumper, Connector_PinHeader_2.54mm:PinHeader_1x02_P2.54mm_Vertical, symbol Jumper:Jumper_2_Open
- added R29, R30, R32, R33, R34: 4.7k, AA_Custom_Components:R_SS_Axial_DIN0207_L6.3mm_D2.5mm_P10.16mm_Horizontal, symbol Device:R
- added TP1: 5V PAD, AA_Custom_Components:TestPoint_Pad_5.0x5.0mm, symbol Connector:TestPoint_Small
- added TP2: GND PAD, AA_Custom_Components:TestPoint_Pad_5.0x5.0mm, symbol Connector:TestPoint_Small
- added TP3: 3.3V PAD, AA_Custom_Components:TestPoint_Pad_5.0x5.0mm, symbol Connector:TestPoint_Small
- added U1: LTC4311, Silicon-Standard:SC70-6, symbol AA_Custom_Components:LTC4311
- JP2: renamed from JP1; footprint AA_Custom_Components:R_SS_Axial_DIN0207_L6.3mm_D2.5mm_P10.16mm_Horizontal -> Connector_PinHeader_2.54mm:PinHeader_1x02_P2.54mm_Vertical
- JP3: footprint AA_Custom_Components:R_SS_Axial_DIN0207_L6.3mm_D2.5mm_P10.16mm_Horizontal -> Connector_PinHeader_2.54mm:PinHeader_1x02_P2.54mm_Vertical
- R27: renamed from R7; footprint Resistor_SMD:R_0603_1608Metric -> AA_Custom_Components:R_SS_Axial_DIN0207_L6.3mm_D2.5mm_P10.16mm_Horizontal; JLCPCB Part # C23162 -> (none)
- U4: renamed from U5; value DFR0753_5V_BUCK -> DFR0753 5V BUCK; footprint (none) -> AA_Custom_Components:DFR0753
- renumbered C7 to C3, C8 to C4, C3 to C5, C10 to C6, C9 to C7, C1 to C8, J4 to J1, J3 to J4, N4 to N1, N3 to N2, R24 to R1, R11 to R10, R14 to R11, R15 to R12, R33 to R13, R34 to R14, R35 to R15, R36 to R16, R2 to R17, R19 to R18, R18 to R19, R13 to R2, R17 to R20, R16 to R21, R25 to R22, R26 to R23, R27 to R24, R28 to R25, R4 to R26, R5 to R28, R12 to R3, R6 to R31, R23 to R4, R1 to R5, R3 to R6, R8 to R7, R9 to R8, R10 to R9, U6 to U2, U1 to U3, U to U5, U3 to U6, U2 to U7, U4 to U8
Connections:
- net +3.3V: now also JP1.1 (A), JP6.2 (B), JP7.2 (B), JP8.2 (B), R29.1, R30.1, R32.1, R33.1, R34.1; no longer C5.1, R1.2, R13.2, R14.2, R15.2, R16.2, R2.2, R22.2, R23.2, R24.2, R25.2, R3.2, R4.2, U3.16 (VPU), U3.4 (VS), U7.16 (VPU), U7.4 (VS), U8.16 (VPU), U8.4 (VS)
- net 2S_BATT_FRONT_CELL1: now also J7.2 (1S)
- net 2S_BATT_FRONT_CELL2: now also J7.3 (2S)
- net 2S_BATT_REAR_CELL1: now also J6.2 (1S)
- net 2S_BATT_REAR_CELL2: now also J6.3 (2S)
- net 3S_BATT_CELL1: now also J5.2 (1S)
- net 3S_BATT_CELL2: now also J5.3 (2S)
- net 3S_BATT_CELL3: now also J5.4 (3S)
- net GND: now also C1.1, C10.2, C9.2, J5.1 (GND), J6.1 (GND), J7.1 (GND), U1.2 (GND), U1.5 (GND)
- net SCL_{1}: now also JP5.1 (A), R29.2; no longer U6.26 (SCL)
- net SCL_{2}: now also R32.2
- net SDA_{1}: now also JP4.1 (A); no longer U6.27 (SDA)
- net SDA_{2}: now also R30.2
- new net: C9.1, JP7.1 (A), R13.2, R14.2, R15.2, R16.2, U7.16 (VPU), U7.4 (VS)
- new net: JP5.2 (C), U6.26 (SCL)
- new net: C1.2, JP1.2 (B), U1.1 (VCC), U1.3 (ENABLE)
- new net: C10.1, JP8.1 (A), R22.2, R23.2, R24.2, R25.2, U8.16 (VPU), U8.4 (VS)
- new net: C5.1, JP6.1 (A), R1.2, R2.2, R3.2, R4.2, U3.16 (VPU), U3.4 (VS)
- new net: J2.1, J3.1
- new net: J2.2, J3.2
- new net: J2.3, J3.3
- new net: JP4.2 (C), U6.27 (SDA)
- new net SCL_{3}: JP5.3 (B), R34.2, U1.6 (BUS1)
- new net SDA_{3}: JP4.3 (B), R33.2, U1.4 (BUS2)
- no-connect marks 18 -> 35
Other:
- note added: "BUZZER"
- note added: "I2C Extender"
- note added: "Jetson (Bus 3) likely has pullup resistors These are Axial Resistors, for ease of switching bus speeds"
- note removed: "TODO: add caps?"
- note removed: "Unsure if Jetson (I2C1) has pullup resistors TODO: Could add extra DNP resistors to change speed?"
- moved on the sheet: BZ1, C8, D1, D2, D3, H1, H2, H3, H4, J1, J4, JP3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

Commit message: Complete Schematic - Add STM32
Parts:
- removed BZ1: Buzzer, AA_Custom_Components:Buzzer_Generic_D12.2mm_H6.5mm, symbol Device:Buzzer
- removed C1: 100nF, Capacitor_SMD:C_0603_1608Metric, symbol Device:C
- removed H1, H2, H3, H4: MountingHole, MountingHole:MountingHole_3.2mm_M3_Pad, symbol Mechanical:MountingHole
- removed J1: GPIO_DEBUG_HEADER, AA_Custom_Components:RASPBERRYPI-40-PIN-GPIO-2x20_P2.54mm_Vertical, symbol AA_Custom_Components:RASPBERRYPI-40-PIN-GPIO
- removed J2: 5V Select Socket, Connector_PinSocket_2.54mm:PinSocket_1x03_P2.54mm_Vertical, symbol dk_Rectangular-Connectors-Headers-Male-Pins:640456-3
- removed J3: 5V Select Jumper, digikey-footprints:PinHeader_1x3_P2.54_Drill1.1mm, symbol dk_Rectangular-Connectors-Headers-Male-Pins:640456-3
- removed J4: Keyed Connector 20 pos, AA_Custom_Components:SULLINS_SFH11-PBPC-D10-ST-BK, symbol AA_Custom_Components:20PosKeyedMale
- removed J5, J6, J7: LIPO_VOLTAGE_ALARM, AA_Custom_Components:LIPO_VOLTAGE_ALARM, symbol AA_Custom_Components:LIPO_VOLTAGE_ALARM
- removed JP1: I2C Extend Jumper, Connector_PinHeader_2.54mm:PinHeader_1x02_P2.54mm_Vertical, symbol Jumper:Jumper_2_Open
- removed JP4: I2C Select SDA, Connector_PinHeader_2.54mm:PinHeader_1x03_P2.54mm_Vertical, symbol Jumper:Jumper_3_Bridged12
- removed JP5: I2C Select SCL, Connector_PinHeader_2.54mm:PinHeader_1x03_P2.54mm_Vertical, symbol Jumper:Jumper_3_Bridged12
- removed N1: ORION LOGO, AA_Custom_Components:Polarity_Center_Positive_7.5mm_SilkScreen, symbol Mechanical:Housing
- removed N2: KiCad, Symbol:KiCad-Logo2_8mm_SilkScreen, symbol Mechanical:Housing
- removed R30, R32: 4.7k, AA_Custom_Components:R_SS_Axial_DIN0207_L6.3mm_D2.5mm_P10.16mm_Horizontal, symbol Device:R
- removed TP1: 5V PAD, AA_Custom_Components:TestPoint_Pad_5.0x5.0mm, symbol Connector:TestPoint_Small
- removed TP2: GND PAD, AA_Custom_Components:TestPoint_Pad_5.0x5.0mm, symbol Connector:TestPoint_Small
- removed TP3: 3.3V PAD, AA_Custom_Components:TestPoint_Pad_5.0x5.0mm, symbol Connector:TestPoint_Small
- removed U1: LTC4311, Silicon-Standard:SC70-6, symbol AA_Custom_Components:LTC4311
- removed U5: NUCLEO64_ARDUINO_UNO_HEADERS, symbol AA_Custom_Components:NUCLEO64_ARDUINO_UNO_HEADERS
- added D4: USB 5V, LED_SMD:LED_0805_2012Metric, symbol Device:LED
- added J1: CONN_20_POS_KEYED_SOCKET, AA_Custom_Components:SULLINS_SBH11-PBPC-D10-ST-BK_SOCKET, symbol AA_Custom_Components:CONN_20_POS_KEYED_SOCKET
- added R35: 470, Resistor_SMD:R_0603_1608Metric, symbol Device:R
- D1: value 5V Buck -> Buck 5V
- D2: value 3.3V STM32 -> STM32 3.3V
- D3: value DEBUG STM32 -> DEBUG
- JP1: renamed from JP2; footprint Connector_PinHeader_2.54mm:PinHeader_1x02_P2.54mm_Vertical -> AA_Custom_Components:Jumper_PinHeader_1x02_P2.54mm_Vertical
- JP2: renamed from JP6; footprint Connector_PinHeader_2.54mm:PinHeader_1x02_P2.54mm_Vertical -> AA_Custom_Components:Jumper_PinHeader_1x02_P2.54mm_Vertical
- JP3: renamed from JP7; footprint Connector_PinHeader_2.54mm:PinHeader_1x02_P2.54mm_Vertical -> AA_Custom_Components:Jumper_PinHeader_1x02_P2.54mm_Vertical
- JP4: renamed from JP3; footprint Connector_PinHeader_2.54mm:PinHeader_1x02_P2.54mm_Vertical -> AA_Custom_Components:Jumper_PinHeader_1x02_P2.54mm_Vertical
- JP7: renamed from JP8; footprint Connector_PinHeader_2.54mm:PinHeader_1x02_P2.54mm_Vertical -> AA_Custom_Components:Jumper_PinHeader_1x02_P2.54mm_Vertical
- U3: renamed from U4; Digikay Part Number (none) -> 1738-DFR0753-ND
- Y1: JLCPCB Part # C97606 -> C32346
- renumbered C2 to C1, C3 to C2, C4 to C3, C5 to C4, C6 to C5, C7 to C6, C8 to C7, C9 to C8, C10 to C9, U2 to U1, U3 to U2, U6 to U4, U7 to U5, U8 to U6
Connections:
- net 2S_BATT_FRONT_CELL1: now also J1.18
- net 2S_BATT_FRONT_CELL2: now also J1.20
- net 2S_BATT_REAR_CELL1: now also J1.14
- net 2S_BATT_REAR_CELL2: now also J1.16
- net 3S_BATT_CELL1: now also J1.13
- net 3S_BATT_CELL2: now also J1.15
- net 3S_BATT_CELL3: now also J1.17
- net GND: now also J1.19, R35.2
- net PWM0: now also J1.1
- net PWM1: now also J1.2
- net PWM10: now also J1.11
- net PWM11: now also J1.12
- net PWM2: now also J1.3
- net PWM3: now also J1.4
- net PWM4: now also J1.5
- net PWM5: now also J1.6
- net PWM6: now also J1.7
- net PWM7: now also J1.8
- net PWM8: now also J1.9
- net PWM9: now also J1.10
- net SCL_{1}: now also U4.26 (SCL)
- net SCL_{2}: no longer U1.19 (COM1)
- net SCL_{3}: now also U1.19 (COM1)
- net SDA_{1}: now also U4.27 (SDA)
- net SDA_{2}: no longer U1.20 (COM0)
- net SDA_{3}: now also U1.20 (COM0)
- new net: D4.1 (K), R35.1
- new net +USB_5V: D4.2 (A)
- no-connect marks 35 -> 17
Other:
- added sheet Compute (Compute.kicad_sch)
- note added: "ORION-CONTROL BOARD"
- note added: "Through-hole Resistors, for ease of tuning bus speeds"
- note removed: "BUZZER"
- note removed: "I2C Extender"
- note removed: "Jetson (Bus 3) likely has pullup resistors These are Axial Resistors, for ease of switching bus speeds"
- note removed: "MOUNTING HARDWARE"
- note removed: "NUCLEO64, IMU, OLED"
- note removed: "Nucleo-F401RE"
- note removed: "ORION - CONTROL BOARD"
- note removed: "PCB LOGOS"
- note removed: "Try to use 0603 (1608m) everywhere. Not smaller."
- moved on the sheet: D2, D3, R28, R31, R33, R34

Commit message: Update JLCPCB rules
Parts:
- removed JP1: BNO Jumper, AA_Custom_Components:Jumper_PinHeader_1x02_P2.54mm_Vertical, symbol Jumper:Jumper_2_Open
- removed JP2: V_{Sense1} Jumper, AA_Custom_Components:Jumper_PinHeader_1x02_P2.54mm_Vertical, symbol Jumper:Jumper_2_Open
- removed JP3: V_{Sense2} Jumper, AA_Custom_Components:Jumper_PinHeader_1x02_P2.54mm_Vertical, symbol Jumper:Jumper_2_Open
- removed JP4: PCA Jumper, AA_Custom_Components:Jumper_PinHeader_1x02_P2.54mm_Vertical, symbol Jumper:Jumper_2_Open
- removed JP7: V_{Sense3} Jumper, AA_Custom_Components:Jumper_PinHeader_1x02_P2.54mm_Vertical, symbol Jumper:Jumper_2_Open
- added JP1: BNO Jumper, AA_Custom_Components:Jumper_PinHeader_1x02_P2.54mm_Vertical, symbol Jumper:Jumper_2_Bridged
- added JP2: VSense1 Jumper, AA_Custom_Components:Jumper_PinHeader_1x02_P2.54mm_Vertical, symbol Jumper:Jumper_2_Bridged
- added JP3: VSense2 Jumper, AA_Custom_Components:Jumper_PinHeader_1x02_P2.54mm_Vertical, symbol Jumper:Jumper_2_Bridged
- added JP4: PCA Jumper, AA_Custom_Components:Jumper_PinHeader_1x02_P2.54mm_Vertical, symbol Jumper:Jumper_2_Bridged
- added JP7: VSense3 Jumper, AA_Custom_Components:Jumper_PinHeader_1x02_P2.54mm_Vertical, symbol Jumper:Jumper_2_Bridged
- Y1: footprint CRYSTAL-SMD-3.2X1.5MM -> Clocks:CRYSTAL-SMD-3.2X1.5MM
Connections:
- net +3.3V: now also JP1.2 (B), JP2.2 (B), JP3.2 (B), JP4.2 (B), JP7.2 (B)
- net at C8.1, R13.2, R14.2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: now also JP3.1 (A)
- net at C1.2, C2.1, U1.28 (VDDIO)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: now also JP1.1 (A)
- net at C9.1, R22.2, R23.2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: now also JP7.1 (A)
- net at C7.2, U4.28 (VDD): now also JP4.1 (A)
- net at C4.1, R1.2, R2.2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: now also JP2.1 (A)
