File: pcb/Orion-Control-Board/Orion-Control-Board.kicad_sch (KiCad schematic)
At the start: 59 parts, among them J1 CONN_20_POS_KEYED_SOCKET, U1 BNO055, U2 INA3221, U3 DFR0753 5V BUCK, U4 PCA9685_PWM_SERVO_DRIVER_IC, U5 INA3221, U6 INA3221, Y1 32.768 kHz

Commit message: Finalize Fab outputs
Parts:
- J1, JP1, JP2, JP3, JP4, JP7, R27, R29, R33, R34: now not fitted
- R10, R11, R12, R18, R19, R20, R21, R5, R6, R7, R8, R9: JLCPCB Part # C25804 -> C22962
- U1: FT Rotation Offset (none) -> -90; ReferenceSchematic https://cdn-learn.adafruit.com/assets/assets/000/024/546/or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 -> (none)
- U3: Digikay Part Number 1738-DFR0753-ND -> (none); Digikey Part # (none) -> 1738-DFR0753-ND; now not fitted
- U4: FT Rotation Offset (none) -> 90

Commit message: Add screen step model
Parts:
- J1, JP1, JP2, JP3, JP4, JP7, R27, R29, R33, R34, U3: now fitted
Changed lines of the file:
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@@
 		(in_bom yes)
 		(on_board yes)
-		(dnp yes)
+		(dnp no)
 		(fields_autoplaced yes)
 		(property "Reference" "JP1"
@@
 		(in_bom yes)
 		(on_board yes)
-		(dnp yes)
+		(dnp no)
 		(property "Reference" "R33"
 			(at 226.822 42.418 0)
@@
 		(in_bom yes)
 		(on_board yes)
-		(dnp yes)
+		(dnp no)
 		(fields_autoplaced yes)
 		(property "Reference" "J1"
@@
 		(in_bom yes)
 		(on_board yes)
-		(dnp yes)
+		(dnp no)
 		(property "Reference" "JP2"
 			(at 57.15 105.41 0)
@@
 		(in_bom yes)
 		(on_board yes)
-		(dnp yes)
+		(dnp no)
 		(property "Reference" "R27"
 			(at 201.422 42.418 0)
@@
 		(in_bom yes)
 		(on_board yes)
-		(dnp yes)
+		(dnp no)
 		(property "Reference" "U3"
 			(at 60.96 164.846 0)
@@
 		(in_bom yes)
 		(on_board yes)
-		(dnp yes)
+		(dnp no)
 		(property "Reference" "R34"
 			(at 234.442 42.418 0)
@@
 		(in_bom yes)
 		(on_board yes)
-		(dnp yes)
+		(dnp no)
 		(property "Reference" "JP3"
 			(at 133.35 105.41 0)
@@
 		(in_bom yes)
 		(on_board yes)
-		(dnp yes)
+		(dnp no)
 		(fields_autoplaced yes)
 		(property "Reference" "JP4"
@@
 		(in_bom yes)
 		(on_board yes)
-		(dnp yes)
+		(dnp no)
 		(property "Reference" "R29"
 			(at 209.042 42.418 0)
@@
 		(in_bom yes)
 		(on_board yes)
-		(dnp yes)
+		(dnp no)
 		(property "Reference" "JP7"
 			(at 207.01 105.41 0)

Commit message: Schematic note
Other:
- note added: "I2C Addr: 0x40"
- note added: "On seperate I2C bus to ensure uninterrupted communication"
- note removed: "12-bit PWM driver I2C Addr: 0x40"
Changed lines of the file:
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@@
 	(text "Through-hole Resistors, for ease of tuning bus speeds"
 		(exclude_from_sim no)
-		(at 184.15 57.15 0)
+		(at 198.882 56.896 0)
 		(effects
 			(font
@@
 		(exclude_from_sim no)
 		(at 107.95 152.654 0)
+		(effects
+			(font
+				(size 1.016 1.016)
+			)
+			(justify left bottom)
+		)
+	)
+	(text "On seperate I2C bus to \nensure uninterrupted communication"
+		(exclude_from_sim no)
+		(at 150.114 53.594 0)
 		(effects
 			(font
@@
 		)
 	)
-	(text "12-bit PWM driver\nI2C Addr: 0x40"
+	(text "I2C Addr: 0x40"
 		(exclude_from_sim no)
 		(at 113.284 84.328 0)

Commit message: Update schematics
Other:
- note added: "CONTROL BOARD"
- note removed: "ORION-CONTROL BOARD"
