File: pcb/Orion-Control-Board/Orion-Control-Board.kicad_pcb (KiCad board)
At the start: 2 copper layers, 70 x 82.4 mm, 87 parts, among them J1 CONN_20_POS_KEYED_SOCKET, J10 POWER, J2 NUCLEO64_CN7, J3 JETSON_ORIN_NANO_DEVKIT_GPIO, J4 5V Select Socket, J5 5V Select Jumper, J6 NUCLEO64_CN10, J7 I2C 1, J8 I2C 3, J9 UART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

Commit message: Finish Control board
Parts:
- added kibuzzard-693F6234: G***, kibuzzard-693F6234, F.Cu at (109.0, 151.0)
- moved R24 50.8 mm to (126.4, 138.6)
- moved R25 50.2 mm to (126.3, 145.8)
- moved R23 45.7 mm to (121.7, 140.2), turned to 180 degrees
- moved R14 43.6 mm to (135.4, 140.2), turned to 180 degrees
- moved JP7 43.4 mm to (121.7, 144.7)
- moved R22 43.4 mm to (121.8, 141.9), turned to 180 degrees
- moved C9 43.4 mm to (130.4, 142.1)
- moved U6 43.4 mm to (126.4, 142.2)
- moved R15 43.2 mm to (140.0, 138.5)
- moved R13 43.0 mm to (135.4, 141.8), turned to 180 degrees
- moved R16 42.4 mm to (139.9, 145.8)
- moved JP3 41.7 mm to (135.3, 144.8)
- moved U5 41.7 mm to (140.0, 142.2)
- moved C8 41.6 mm to (143.9, 141.9)
- moved JP1 8.62 mm to (148.2, 137.6), turned to -90 degrees
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Routing:
- net SDA_{3}: track 57.9 -> 120.1 mm, vias 0 -> 7
- net SCL_{3}: track 56.2 -> 112.7 mm, vias 3 -> 5
- net 3S_BATT_CELL1: track 48.3 -> 103.1 mm, vias 0 -> 4
- net 3S_BATT_CELL2: track 49.0 -> 97.3 mm, vias 0 -> 4
- net 2S_BATT_FRONT_CELL1: track 67.8 -> 115.3 mm, vias 2 -> 6
- net 3S_BATT_CELL3: track 49.9 -> 95.8 mm, vias 0 -> 4
- net 2S_BATT_REAR_CELL1: track 50.8 -> 95.8 mm, vias 0 -> 4
- net 2S_BATT_REAR_CELL2: track 51.1 -> 91.3 mm, vias 0 -> 4
- net Net-(JP7-A): track 0.00 -> 27.7 mm
- net Net-(JP3-A): track 0.00 -> 26.4 mm
- net GND: track 84.1 -> 95.6 mm, vias 29 -> 31
- net +3.3V: track 6.30 -> 11.1 mm, vias 2 -> 4
- net 2S_BATT_FRONT_CELL2: track 117.0 -> 119.9 mm, vias 2 -> 4
- net Net-(U6-CRITICAL): track 0.00 -> 2.86 mm
- net Net-(U5-CRITICAL): track 0.00 -> 2.72 mm
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Other:
- board text added: "By: Ashish Agrahari"
