File: pcb/Orion-Control-Board/Orion-Control-Board.kicad_pcb (KiCad board)
At the start: 2 copper layers, 70 x 82.4 mm, 88 parts, among them J1 CONN_20_POS_KEYED_SOCKET, J10 POWER, J2 NUCLEO64_CN7, J3 JETSON_ORIN_NANO_DEVKIT_GPIO, J4 5V Select Socket, J5 5V Select Jumper, J6 NUCLEO64_CN10, J7 I2C 1, J8 I2C 3, J9 UART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

Commit message: Review Power board.
Other:
- board text added: "JLCJLCJLCJLC"
Changed lines of the file:
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@@
+		)
+	)
+	(gr_text "JLCJLCJLCJLC"
+		(at 122.075 151.7 0)
+		(layer "B.SilkS")
+		(effects
+			(font
+				(size 1 1)
+				(thickness 0.153)
+			)
+			(justify left bottom mirror)
 		)
 	)
