Commit message: Fix urdf limits and upadte launch

File: Software/Jetson/workspace/isaac_ros-dev/src/orion_urdf/urdf/robot_description.urdf (robot description, URDF)
Before this commit: robot orion_urdf, 17 links, 16 joints
Joints:
- joint back_left_joint_1: limit lower=0 upper=0 effort=0 velocity=0 -> lower=-3.14159 upper=3.14159 effort=10.0 velocity=1.0
- joint back_left_joint_2: limit lower=0 upper=0 effort=0 velocity=0 -> lower=-3.14159 upper=3.14159 effort=10.0 velocity=1.0
- joint back_left_joint_3: limit lower=0 upper=0 effort=0 velocity=0 -> lower=-3.14159 upper=3.14159 effort=10.0 velocity=1.0
- joint back_right_joint_1: limit lower=0 upper=0 effort=0 velocity=0 -> lower=-3.14159 upper=3.14159 effort=10.0 velocity=1.0
- joint back_right_joint_2: limit lower=0 upper=0 effort=0 velocity=0 -> lower=-3.14159 upper=3.14159 effort=10.0 velocity=1.0
- joint back_right_joint_3: limit lower=0 upper=0 effort=0 velocity=0 -> lower=-3.14159 upper=3.14159 effort=10.0 velocity=1.0
- joint front_left_joint_1: limit lower=0 upper=0 effort=0 velocity=0 -> lower=-3.14159 upper=3.14159 effort=10.0 velocity=1.0
- joint front_left_joint_2: limit lower=0 upper=0 effort=0 velocity=0 -> lower=-3.14159 upper=3.14159 effort=10.0 velocity=1.0
- joint front_left_joint_3: limit lower=0 upper=0 effort=0 velocity=0 -> lower=-3.14159 upper=3.14159 effort=10.0 velocity=1.0
- joint front_right_joint_1: limit lower=0 upper=0 effort=0 velocity=0 -> lower=-3.14159 upper=3.14159 effort=10.0 velocity=1.0
- joint front_right_joint_2: limit lower=0 upper=0 effort=0 velocity=0 -> lower=-3.14159 upper=3.14159 effort=10.0 velocity=1.0
- joint front_right_joint_3: limit lower=0 upper=0 effort=0 velocity=0 -> lower=-3.14159 upper=3.14159 effort=10.0 velocity=1.0

Commit message: Remove old urdf

File: Software/Jetson/workspace/isaac_ros-dev/src/orion_urdf/urdf/robot_description.urdf (robot description, URDF)
Before this commit: robot orion_urdf, 17 links, 16 joints
Links:
- removed link lidar_link
- added link laser, mass 0.073251; collision mesh filename=package://orion_urdf/meshes/lidar_link.STL; visual mesh filename=package://orion_urdf/meshes/lidar_link.STL
- added link lid_link, mass 0.47342; collision mesh filename=package://orion_urdf/meshes/lid_link.STL; visual mesh filename=package://orion_urdf/meshes/lid_link.STL
- link back_left_link_1: mass 0.110718200835103 -> 0.11072
- link back_left_link_2: mass 0.0652435231118066 -> 0.065244
- link back_left_link_3: mass 0.0592549511706032 -> 0.052056
- link back_right_link_1: mass 0.1107181974716 -> 0.11072
- link back_right_link_2: mass 0.0652435283702889 -> 0.065244
- link back_right_link_3: mass 0.0592586186370103 -> 0.05206
- link chassis_link: mass 1.7618 -> 1.2884
- link front_left_link_1: mass 0.110718199912909 -> 0.11072
- link front_left_link_2: mass 0.0652435230220067 -> 0.065244
- link front_left_link_3: mass 0.0592549516376399 -> 0.052056
- link front_right_link_1: mass 0 -> 0.14335
- link front_right_link_2: mass 0.065243528810921 -> 0.065244
- link front_right_link_3: mass 0.0592586215672063 -> 0.05206
- link left_camera_link: mass 0.00432134882914042 -> 0.0043213
- link right_camera_link: mass 0.00432566682914042 -> 0.0043257
Joints:
- added joint lid_joint: type fixed, parent chassis_link, child lid_link, origin xyz=0.01 0 0.1 rpy=0 0 0, axis 0 0 0
- joint back_left_joint_1: limit lower=-3.14159 upper=3.14159 effort=10.0 velocity=1.0 -> lower=-3.1416 upper=3.1416 effort=10 velocity=1; origin xyz=0.01225 -0.33471 0.045907 rpy=0.0031593 0 1.5708 -> xyz=-0.134705178168527 0.082750000000001 0.0459074375810237 rpy=0.00315930390260669 0 0
- joint back_left_joint_2: limit lower=-3.14159 upper=3.14159 effort=10.0 velocity=1.0 -> lower=-3.1416 upper=3.1416 effort=10 velocity=1; origin xyz=0 0.0392977405875028 0.000624999999996156 rpy=0 0 0 -> xyz=0 0.0392977405875036 0.000624999999999577 rpy=0 0 0
- joint back_left_joint_3: limit lower=-3.14159 upper=3.14159 effort=10.0 velocity=1.0 -> lower=-3.1416 upper=3.1416 effort=10 velocity=1; origin xyz=-0.0969291533452488 0 -0.0509410368148632 rpy=0 0 0 -> xyz=-0.0969291533452496 0 -0.0509410368148617 rpy=0 0 0
- joint back_right_joint_1: limit lower=-3.14159 upper=3.14159 effort=10.0 velocity=1.0 -> lower=-3.1416 upper=3.1416 effort=10 velocity=1; origin xyz=0.17745 -0.33471 0.045907 rpy=-0.02534 0 1.5708 -> xyz=-0.134705178168499 -0.0824499999999989 0.0459074375810237 rpy=-0.0253401254512525 0 0
- joint back_right_joint_2: limit lower=-3.14159 upper=3.14159 effort=10.0 velocity=1.0 -> lower=-3.1416 upper=3.1416 effort=10 velocity=1; origin xyz=0 -0.039297740587504 0.000624999999998224 rpy=0 0 0 -> xyz=0 -0.0392977405875037 0.000625000000000271 rpy=0 0 0
- joint back_right_joint_3: limit lower=-3.14159 upper=3.14159 effort=10.0 velocity=1.0 -> lower=-3.1416 upper=3.1416 effort=10 velocity=1; origin xyz=-0.0914299430637919 0 -0.0602562639263626 rpy=0 0 0 -> xyz=-0.0914299430637917 0 -0.0602562639263631 rpy=0 0 0
- joint front_left_joint_1: limit lower=-3.14159 upper=3.14159 effort=10.0 velocity=1.0 -> lower=-3.1416 upper=3.1416 effort=10 velocity=1; origin xyz=0.01255 -0.08621 0.045907 rpy=0.0046679 0 1.5708 -> xyz=0.113790303006481 0.0824500000000011 0.0459074375810237 rpy=0.00466787437143287 0 0
- joint front_left_joint_2: limit lower=-3.14159 upper=3.14159 effort=10.0 velocity=1.0 -> lower=-3.1416 upper=3.1416 effort=10 velocity=1; origin xyz=0 0.0392977405875039 0.000624999999998176 rpy=0 0 0 -> xyz=0 0.0392977405875036 0.000624999999999681 rpy=0 0 0
- joint front_left_joint_3: limit lower=-3.14159 upper=3.14159 effort=10.0 velocity=1.0 -> lower=-3.1416 upper=3.1416 effort=10 velocity=1; origin xyz=-0.0969291533452484 0 -0.0509410368148641 rpy=0 0 0 -> xyz=-0.0969291533452496 0 -0.0509410368148619 rpy=0 0 0
- joint front_right_joint_1: limit lower=-3.14159 upper=3.14159 effort=10.0 velocity=1.0 -> lower=-3.1416 upper=3.1416 effort=10 velocity=1; origin xyz=0.177749999999999 -0.0862096969935193 0.0459074375810233 rpy=-0.0196130777187637 0 1.5707963267949 -> xyz=0.113790303006509 -0.0827499999999989 0.0459074375810237 rpy=-0.0196130777187636 0 0
- joint front_right_joint_2: limit lower=-3.14159 upper=3.14159 effort=10.0 velocity=1.0 -> lower=-3.1416 upper=3.1416 effort=10 velocity=1; origin xyz=0 -0.0392977405875036 0.000625000000000368 rpy=0 0 0 -> xyz=0 -0.0392977405875038 0.000624999999999792 rpy=0 0 0
- joint front_right_joint_3: limit lower=-3.14159 upper=3.14159 effort=10.0 velocity=1.0 -> lower=-3.1416 upper=3.1416 effort=10 velocity=1; origin xyz=-0.0914299430637918 0 -0.0602562639263623 rpy=0 0 0 -> xyz=-0.0914299430637918 0 -0.0602562639263629 rpy=0 0 0
- joint left_camera_joint: origin xyz=0.06515 -0.01347 0.09735 rpy=0 0 1.5708 -> xyz=0.18653 0.02985 0.09735 rpy=0 0 0
- joint lidar_joint: child lidar_link -> laser; origin xyz=0.095089 -0.086952 0.1345 rpy=0 0 1.5708 -> xyz=0.11305 -8.8769E-05 0.1345 rpy=0 0 3.14159
- joint right_camera_joint: origin xyz=0.125249999999999 -0.0134698446791103 0.0973500000000002 rpy=0 0 1.5707963267949 -> xyz=0.18653 -0.03025 0.09735 rpy=0 0 0

Commit message: Fix urdf to have proper angles from stm

File: Software/Jetson/workspace/isaac_ros-dev/src/orion_urdf/urdf/robot_description.urdf (robot description, URDF)
Before this commit: robot orion_urdf, 18 links, 17 joints
Joints:
- joint back_left_joint_1: limit lower=-3.1416 upper=3.1416 effort=10 velocity=1 -> lower=-3.1416 upper=3.1416 effort=1000 velocity=100; origin xyz=-0.134705178168527 0.082750000000001 0.0459074375810237 rpy=0.00315930390260669 0 0 -> xyz=-0.134705178168527 0.082750000000001 0.0459074375810237 rpy=0 0 0
- joint back_left_joint_2: limit lower=-3.1416 upper=3.1416 effort=10 velocity=1 -> lower=-3.1416 upper=3.1416 effort=1000 velocity=100
- joint back_left_joint_3: limit lower=-3.1416 upper=3.1416 effort=10 velocity=1 -> lower=-3.1416 upper=3.1416 effort=1000 velocity=100
- joint back_right_joint_1: limit lower=-3.1416 upper=3.1416 effort=10 velocity=1 -> lower=-3.1416 upper=3.1416 effort=1000 velocity=100; origin xyz=-0.134705178168499 -0.0824499999999989 0.0459074375810237 rpy=-0.0253401254512525 0 0 -> xyz=-0.134705178168499 -0.0824499999999989 0.0459074375810237 rpy=0 0 0
- joint back_right_joint_2: limit lower=-3.1416 upper=3.1416 effort=10 velocity=1 -> lower=-3.1416 upper=3.1416 effort=1000 velocity=100
- joint back_right_joint_3: limit lower=-3.1416 upper=3.1416 effort=10 velocity=1 -> lower=-3.1416 upper=3.1416 effort=1000 velocity=100
- joint chassis_joint: origin (none) -> xyz=0 0 0.07 rpy=0 0 0
- joint front_left_joint_1: limit lower=-3.1416 upper=3.1416 effort=10 velocity=1 -> lower=-3.1416 upper=3.1416 effort=1000 velocity=100; origin xyz=0.113790303006481 0.0824500000000011 0.0459074375810237 rpy=0.00466787437143287 0 0 -> xyz=0.113790303006481 0.0824500000000011 0.0459074375810237 rpy=0 0 0
- joint front_left_joint_2: limit lower=-3.1416 upper=3.1416 effort=10 velocity=1 -> lower=-3.1416 upper=3.1416 effort=1000 velocity=100
- joint front_left_joint_3: limit lower=-3.1416 upper=3.1416 effort=10 velocity=1 -> lower=-3.1416 upper=3.1416 effort=1000 velocity=100
- joint front_right_joint_1: limit lower=-3.1416 upper=3.1416 effort=10 velocity=1 -> lower=-3.1416 upper=3.1416 effort=1000 velocity=100; origin xyz=0.113790303006509 -0.0827499999999989 0.0459074375810237 rpy=-0.0196130777187636 0 0 -> xyz=0.113790303006509 -0.0827499999999989 0.0459074375810237 rpy=0 0 0
- joint front_right_joint_2: limit lower=-3.1416 upper=3.1416 effort=10 velocity=1 -> lower=-3.1416 upper=3.1416 effort=1000 velocity=100
- joint front_right_joint_3: limit lower=-3.1416 upper=3.1416 effort=10 velocity=1 -> lower=-3.1416 upper=3.1416 effort=1000 velocity=100

Commit message: Add in launches

File: Software/Jetson/workspace/isaac_ros-dev/src/orion_urdf/urdf/robot_description.urdf (robot description, URDF)
Before this commit: robot orion_urdf, 18 links, 17 joints
Joints:
- joint chassis_joint: origin xyz=0 0 0.07 rpy=0 0 0 -> xyz=0 0 0.09 rpy=0 0 0
