Commit message: Usd initial tests

File: Software/reinforcement-learning/src/robot_description/robot.urdf (robot description, URDF)
Before this commit: robot quadruped_robot, 21 links, 20 joints
Joints:
- joint FL_calf_joint: limit lower=-3.1416 upper=3.1416 effort=500 velocity=10 -> lower=-0.872665 upper=0.872665 effort=500 velocity=10
- joint FL_hip_joint: limit lower=-3.1416 upper=3.1416 effort=500 velocity=10 -> lower=-0.349066 upper=0.349066 effort=500 velocity=10
- joint FL_thigh_joint: limit lower=-3.1416 upper=3.1416 effort=500 velocity=10 -> lower=-1.22173 upper=0 effort=500 velocity=10
- joint FR_calf_joint: limit lower=-3.1416 upper=3.1416 effort=500 velocity=10 -> lower=-0.872665 upper=0.872665 effort=500 velocity=10
- joint FR_hip_joint: limit lower=-3.1416 upper=3.1416 effort=500 velocity=10 -> lower=-0.349066 upper=0.349066 effort=500 velocity=10
- joint FR_thigh_joint: limit lower=-3.1416 upper=3.1416 effort=500 velocity=10 -> lower=0 upper=1.22173 effort=500 velocity=10
- joint RL_calf_joint: limit lower=-3.1416 upper=3.1416 effort=500 velocity=10 -> lower=-0.872665 upper=0.872665 effort=500 velocity=10
- joint RL_hip_joint: limit lower=-3.1416 upper=3.1416 effort=500 velocity=10 -> lower=-0.349066 upper=0.349066 effort=500 velocity=10
- joint RL_thigh_joint: limit lower=-3.1416 upper=3.1416 effort=500 velocity=10 -> lower=-1.22173 upper=0 effort=500 velocity=10
- joint RR_calf_joint: limit lower=-3.1416 upper=3.1416 effort=500 velocity=10 -> lower=-0.872665 upper=0.872665 effort=500 velocity=10
- joint RR_hip_joint: limit lower=-3.1416 upper=3.1416 effort=500 velocity=10 -> lower=-0.349066 upper=0.349066 effort=500 velocity=10
- joint RR_thigh_joint: limit lower=-3.1416 upper=3.1416 effort=500 velocity=10 -> lower=0 upper=1.22173 effort=500 velocity=10
